File: hardware/hub/v0.1/Mythra-hub/ufp.kicad_sch (KiCad schematic)
At the start: 18 parts, among them J1 918-418K2022C40000, J11 DFP SWD, U2 HD3SS460, U20 CYPD3174-24, U35 SP3400-02UTG

Commit message: Fixed the PD controller footprints so the gnd on pin 22 was hooked up
Parts:
- U20: MFR Cypress -> (property "Reference" "U" (id 0) (at -17.78 21.59 0); MPN CYPD3174-24LQXQ -> (effects (font (size 1.27 1.27)) (justify left)); OC_FARNELL 2896248 -> ); URL_FARNELL https://uk.farnell.com/cypress-semiconductor/cypd3174-24lqx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 -> (property "Value" "CYPD3174-24" (id 1) (at 17.78 -21.59 0)
Connections:
- net GND: now also U20.22 (GND)

Commit message: Fixed some mishaps with the PD controller metadata fields and sync'd the schematic and PCB for the hub
Parts:
- U20: MFR (property "Reference" "U" (id 0) (at -17.78 21.59 0) -> Cypress; MPN (effects (font (size 1.27 1.27)) (justify left)) -> CYPD3174-24LQXQ; OC_FARNELL ) -> 2896248; URL_FARNELL (property "Value" "CYPD3174-24" (id 1) (at 17.78 -21.59 0) -> https://uk.farnell.com/cypress-semiconductor/cypd3174-24lqx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
